Commit message: URDF robots (stream U): Blastoise synced from the real-boat URDF, minimal_boat example, RobotCatalog, UrdfTests
- blastoise.urdf is the expanded real xacro (real gps/imu/props; crane-only ball_dropper/water_pump links
  removed), with its profile (body yaw 90, Blastoise templates). Blastoise.prefab synced from it with every
  GameObject/Transform fileID kept (173/173); it now carries RobotDescription with its geometry hashes, and
  gps_link/imu_link (no <inertial>) go from the importer's 1 kg to 0.001 kg (the plant rescales link masses
  to the profile mass; only the legacy-physics path sees 2 kg less).
- Assets/Robot Descriptions/minimal_boat: an agent-written boat (box hull, two thrusters, lidar), synced
  with the Surface profile; the single copy, used as the test fixture too. Its URDF mass is 20.84 kg and the
  imported boat now weighs that (was 21.84: the massless laser_frame had the importer's 1 kg).
- RobotCatalog: --crane-robot blastoise | minimal_boat.
- UrdfTests: Blastoise matches its URDF, prefab and course-scene boat (CheckScene, 1 mm / 0.1 deg, anchors
  included); a scene anchor override fails the check (text override and the instantiated 10 mm anchor
  offset); lost geometry hashes re-import onto the same objects byte-identically; agent import gets its
  components, re-syncs byte-identically, laser_frame near-zero mass; drive test (alone in an empty scene,
  thrust at CG height since no water rights the hull) checks mass against the URDF's own inertials.

File: Assets/Robot Descriptions/blastoise/blastoise.urdf (robot description, URDF)
Before this commit: robot blastoise, 18 links, 17 joints
Links:
- removed link ball_dropper_link
- removed link water_pump_link
- link base_link: mass 3.00000 -> 10.0; geometry collision box size=0.18120 0.18120 0.18120; collision box size=0.50929 0.43980 0.17333
- link front_camera_link: mass 0.10000 -> None; geometry visual mesh filename=package://mhseals_nav/description/blastoise/meshes/front_ca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
- link front_left_propeller_link: mass 0.01000 -> None; geometry visual mesh filename=package://mhseals_nav/description/blastoise/meshes/front_le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 scale=1 1 1
- link front_left_thruster_link: geometry visual mesh filename=package://mhseals_nav/description/blastoise/meshes/front_le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 scale=1 1 1
- link front_right_propeller_link: mass 0.01000 -> None; geometry visual mesh filename=package://mhseals_nav/description/blastoise/meshes/front_ri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 scale=1 1 1
- link front_right_thruster_link: geometry visual mesh filename=package://mhseals_nav/description/blastoise/meshes/front_ri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 scale=1 1 1
- link left_hull_link: mass 7.00000 -> 9.0; geometry collision mesh filename=package://mhseals_nav/description/blastoise/meshes/left_hul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 scale=0.001 0.001 0.00081; visual mesh filename=package://mhseals_nav/description/blastoise/meshes/left_hul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
- link lidar_link: mass 0.10000 -> None; geometry visual mesh filename=package://mhseals_nav/description/blastoise/meshes/lidar.stl
- link rear_left_propeller_link: mass 0.01000 -> None; geometry visual mesh filename=package://mhseals_nav/description/blastoise/meshes/rear_lef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 scale=1 1 1
- link rear_left_thruster_link: geometry visual mesh filename=package://mhseals_nav/description/blastoise/meshes/rear_lef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 scale=1 1 1
- link rear_right_propeller_link: mass 0.01000 -> None; geometry visual mesh filename=package://mhseals_nav/description/blastoise/meshes/rear_rig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 scale=1 1 1
- link rear_right_thruster_link: geometry visual mesh filename=package://mhseals_nav/description/blastoise/meshes/rear_rig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 scale=1 1 1
- link right_hull_link: mass 7.00000 -> 9.0; geometry collision mesh filename=package://mhseals_nav/description/blastoise/meshes/right_hu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 scale=0.001 0.001 0.00081; visual mesh filename=package://mhseals_nav/description/blastoise/meshes/right_hu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
- link sensor_mount_link: mass 0.30000 -> 0.3
Joints:
- removed joint ball_dropper_joint
- removed joint front_left_propeller_link
- removed joint front_left_thruster_joint
- removed joint front_right_propeller_joint
- removed joint front_right_thruster_joint
- removed joint gps_joint
- removed joint imu_joint
- removed joint rear_left_propeller_link
- removed joint rear_left_thruster_joint
- removed joint rear_right_propeller_joint
- removed joint rear_right_thruster_joint
- removed joint water_pump_joint
- added joint front_left_propeller_link_joint: type fixed, parent front_left_thruster_link, child front_left_propeller_link, origin xyz=0 0 -0.00299
- added joint front_left_thruster_link_joint: type fixed, parent left_hull_link, child front_left_thruster_link, origin xyz=-0.01287 0.26637 -0.28232 rpy=1.57080 0 2.35619
- added joint front_right_propeller_link_joint: type fixed, parent front_right_thruster_link, child front_right_propeller_link, origin xyz=0 0 -0.00299
- added joint front_right_thruster_link_joint: type fixed, parent right_hull_link, child front_right_thruster_link, origin xyz=0.01287 0.26636 -0.28432 rpy=1.57080 0 -2.35619
- added joint gps_link_joint: type fixed, parent base_link, child gps_link, origin xyz=0.051 -0.127 0.23439
- added joint imu_link_joint: type fixed, parent base_link, child imu_link, origin xyz=-0.051 -0.127 0
- added joint rear_left_propeller_link_joint: type fixed, parent rear_left_thruster_link, child rear_left_propeller_link, origin xyz=0 0 -0.00299
- added joint rear_left_thruster_link_joint: type fixed, parent left_hull_link, child rear_left_thruster_link, origin xyz=-0.01277 -0.26625 -0.28232 rpy=1.57080 0 0.78540
- added joint rear_right_propeller_link_joint: type fixed, parent rear_right_thruster_link, child rear_right_propeller_link, origin xyz=0 0 -0.00299
- added joint rear_right_thruster_link_joint: type fixed, parent right_hull_link, child rear_right_thruster_link, origin xyz=0.01282 -0.26630 -0.28432 rpy=1.57080 0 -0.78540
- joint front_camera_joint: origin xyz=0.00000 0.04990 0.13779 rpy=0.00000 0.00000 0.00000 -> xyz=0.04990 0 0.13779 rpy=0 0 0
- joint left_hull_joint: origin xyz=-0.33020 0.00000 -0.08000 rpy=0.00000 0.00000 0.00000 -> xyz=0 0.33020 -0.08000 rpy=0 0 -1.57080
- joint lidar_joint: origin xyz=0.00000 0.01270 0.29035 rpy=0.00000 0.00000 0.00000 -> xyz=0.01270 0 0.29035 rpy=0 0 0
- joint right_hull_joint: origin xyz=0.33020 0.00000 -0.07800 rpy=0.00000 0.00000 0.00000 -> xyz=0 -0.33020 -0.07800 rpy=0 0 -1.57080
- joint sensor_mount_joint: origin xyz=0.00000 0.27711 -0.01260 rpy=0.00000 0.00000 0.00000 -> xyz=0.27711 0 -0.01260 rpy=0 0 0
